Commit message: done

File: urdf_file/my_bot.urdf.xacro (robot description, xacro)
@@ -1,7 +1,15 @@
 <?xml version="1.0"?>
 <robot xmlns:xacro="http://www.ros.org/wiki/xacro"  name="robot">
+    <xacro:arg name="use_ros2_control" default="true"/>
+    <xacro:arg name="sim_mode" default="false"/>
     <xacro:include filename="my_bot_core.xacro" />
-    <xacro:include filename="my_bot_gazebo_control.xacro" />
+    <xacro:include filename="ros2_control.xacro" />
+    <xacro:if value="$(arg use_ros2_control)">
+    </xacro:if>
+    <xacro:unless value="$(arg use_ros2_control)">
+        <xacro:include filename="my_bot_gazebo_control.xacro" />
+    </xacro:unless>
     <xacro:include filename="lidar.xacro" />
     <xacro:include filename="camera1.xacro" />
+    <!-- <xacro:include filename="depth_camera.xacro" /> -->
 </robot>

File: urdf_file/my_bot_core.xacro (robot description, xacro)
@@ -14,5 +14,5 @@
         <color rgba="0 0 0 1"/>
     </material>
-    <xacro:property name="pi" value="3.141592653589793"/>
+    <!--<xacro:property name="pi" value="3.141592653589793"/>-->
     <link name="base_link">
     </link>

File: urdf_file/ros2_control.xacro (robot description, xacro)
@@ -57,5 +57,5 @@
         <plugin name="gazebo_ros2_control" filename="libgazebo_ros2_control.so">
             <parameters>$(find articubot_one)/config/my_controllers.yaml</parameters>
-            <parameters>$(find articubot_one)/config/gaz_ros2_ctl_use_sim.yaml</parameters>
+            <!--<parameters>$(find articubot_one)/config/gaz_ros2_ctl_use_sim.yaml</parameters>-->
         </plugin>
     </gazebo>
