Commit message: Updated launch and URDF files

File: urdf_file/my_bot_core.xacro (robot description, xacro)
@@ -16,4 +16,11 @@
     <xacro:property name="pi" value="3.141592653589793"/>
     <link name="base_link">
+    </link>
+    <joint name="base_footprint_joint" type="fixed">
+        <parent link="base_link"/>
+        <child link="base_footprint"/>
+        <origin xyz="0 0 0" rpy="0 0 0"/>
+    </joint>
+    <link name="base_footprint">
     </link>
     <joint name="chassis_joint" type="fixed">

Commit message: Updated launch and URDF files

File: urdf_file/my_bot_core.xacro (robot description, xacro)
@@ -53,5 +53,5 @@
         <parent link="base_link"/>
         <child link="left_wheel"/>
-        <origin xyz="0 0.175 0" rpy="${pi/2} 0 0"/>
+        <origin xyz="0 0.175 0" rpy="1.57  0 0"/>
         <axis xyz="0 0 -1"/>
     </joint>
@@ -78,5 +78,5 @@
         <parent link="base_link"/>
         <child link="right_wheel"/>
-        <origin xyz="0 -0.175 0" rpy="${pi/2} 0 0"/>
+        <origin xyz="0 -0.175 0" rpy="1.57 0 0"/>
         <axis xyz="0 0 -1"/>
     </joint>

File: urdf_file/ros2_control.xacro (robot description, xacro)
@@ -56,6 +56,6 @@
     <gazebo>
         <plugin name="gazebo_ros2_control" filename="libgazebo_ros2_control.so">
-            <parameters>$(find articubot_one)/config/my_controllers.yaml</parameters>
-            <!--<parameters>$(find articubot_one)/config/gaz_ros2_ctl_use_sim.yaml</parameters>-->
+            <parameters>$(find autobot_pkg)/config/my_controllers.yaml</parameters>
+            <parameters>$(find autobot_pkg)/config/gaz_ros2_ctl_use_sim.yaml</parameters>
         </plugin>
     </gazebo>
